File: tests/assets/non-plated-hole.kicad_pcb (KiCad board)
At the start: 2 copper layers, 50 x 50 mm, 4 parts

Commit message: feat: Dynamically name standalone PCB hole footprints in KiCad based on their shape and dimensions
Parts:
- ? (x2): footprint tscircuit:MountingHole -> tscircuit:hole_circle_3.2mm
Changed lines of the file:
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@@
   )
   (footprint
-    "tscircuit:MountingHole"
+    "tscircuit:hole_circle_3.2mm"
     (layer F.Cu)
     (at 100 100 0)
@@
   )
   (footprint
-    "tscircuit:MountingHole"
+    "tscircuit:hole_circle_3.2mm"
     (layer F.Cu)
     (at 100 100 0)

Commit message: up
Parts:
- ? (x2): footprint tscircuit:hole_circle_3.2mm -> tscircuit:hole_circle_holeDiameter3.2mm
Changed lines of the file:
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@@
   )
   (footprint
-    "tscircuit:hole_circle_3.2mm"
+    "tscircuit:hole_circle_holeDiameter3.2mm"
     (layer F.Cu)
     (at 100 100 0)
@@
   )
   (footprint
-    "tscircuit:hole_circle_3.2mm"
+    "tscircuit:hole_circle_holeDiameter3.2mm"
     (layer F.Cu)
     (at 100 100 0)
