File: tests/assets/repro07-standalone-hole-naming.kicad_pcb (KiCad board)
At the start: 2 copper layers, 50 x 50 mm, 2 parts

Commit message: up
Parts:
- ?: footprint tscircuit:hole_circle_3mm -> tscircuit:hole_circle_holeDiameter3mm
- ?: footprint tscircuit:hole_pill_4mm_2mm -> tscircuit:hole_pill_holeWidth4mm_holeHeight2mm
Changed lines of the file:
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@@
   (net 0 "")
   (footprint
-    "tscircuit:hole_circle_3mm"
+    "tscircuit:hole_circle_holeDiameter3mm"
     (layer F.Cu)
     (at 100 100 0)
@@
   )
   (footprint
-    "tscircuit:hole_pill_4mm_2mm"
+    "tscircuit:hole_pill_holeWidth4mm_holeHeight2mm"
     (layer F.Cu)
     (at 100 100 0)
