File: tests/assets/repro18-rotated-chip-pill-plated-hole.kicad_pcb (KiCad board)
At the start: 2 copper layers, 11 x 11 mm, 1 part

Commit message: up
Parts:
- moved U1 5.00 mm to (101.6, 95.7)
Changed lines of the file:
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@@
     "tscircuit:chip"
     (layer F.Cu)
-    (at 101.57511755 100.675015 -90)
+    (at 101.57511755 95.675015 -90)
     (property "Reference" "U1"
       (at 0 -3 0)
@@
     )
     (pad "13" thru_hole oval
-      (at 0 0 270)
+      (at 0 0 180)
       (size 1.0999978 1.999996)
       (drill oval 0.5999988 1.499997)
