File: tests/assets/repro18-rotated-chip-pill-plated-hole.kicad_pcb (KiCad board)
At the start: 2 copper layers, 11 x 11 mm, 1 part

Commit message: Fall back to the component name for a chip's KiCad Value
`<chip>` was the only component type with no fallback value: a chip
without a manufacturerPartNumber exported as `(property "Value" "")`,
where a resistor falls back to "R", an LED to "LED" and every unhandled
ftype to the component's name.

An empty Value is not just cosmetic. KiCad's Specctra DSN export (used
by the freerouting plugin) refuses the board with "Footprint with value
of '' has an empty reference designator", so a design with a plain
`<chip>` cannot be handed to KiCad's own routing tooling.

Use the name, matching what the function already does for every ftype it
doesn't special-case.
Parts:
- U1: value (none) -> U1
Changed lines of the file:
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@@
       )
     )
-    (property "Value" ""
+    (property "Value" "U1"
       (at 0 3 0)
       (layer F.Fab)
