File: tests/assets/repro18-rotated-chip-pill-plated-hole.kicad_pcb (KiCad board)
At the start: 2 copper layers, 11 x 11 mm, 1 part

Commit message: fix: use importer rotation fix without exporter compensation
Parts:
- turned U1 to -90 degrees
Changed lines of the file:
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@@
     "tscircuit:chip"
     (layer F.Cu)
-    (at 101.57511755 95.675015 90)
+    (at 101.57511755 95.675015 -90)
     (property "Reference" "U1"
       (at 0 -3 0)

Commit message: Handle legacy paste geometry and library export compatibility
Parts:
- added ?: , tscircuit:solder_paste, F.Cu at (101.6, 95.7)
- added ?: , tscircuit:solder_paste, B.Cu at (101.6, 95.7)
Changed lines of the file:
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@@
+    )
+  )
+  (footprint
+    "tscircuit:solder_paste"
+    (layer F.Cu)
+    (at 101.57511755 95.675015 0)
+    (attr board_only exclude_from_pos_files exclude_from_bom)
+    (pad "" smd roundrect
+      (at 0 0 0)
+      (size 1.0999978 1.999996)
+      (layers F.Paste)
+      (roundrect_rratio 0.5)
+    )
+  )
+  (footprint
+    "tscircuit:solder_paste"
+    (layer B.Cu)
+    (at 101.57511755 95.675015 0)
+    (attr board_only exclude_from_pos_files exclude_from_bom)
+    (pad "" smd roundrect
+      (at 0 0 0)
+      (size 1.0999978 1.999996)
+      (layers B.Paste)
+      (roundrect_rratio 0.5)
     )
   )
